Commit message: Temporal fix in the URDF to move the Kinect out of the arm's reach until we calibrate its extrinsic parameters

File: ridgeback_yumi_description/urdf/ridgeback_yumi.urdf (robot description, URDF)
Before this commit: robot ridgeback_yumi, 48 links, 47 joints
Joints:
- joint kinect2_to_left_kinect_base: origin xyz=0.1 0.03 0.56 rpy=0 -0.523598775598 -0.17 -> xyz=-0.1 0.03 0.56 rpy=0 -1.57079632679 -0.17
- joint kinect2_to_right_kinect_base: origin xyz=0.1 -0.03 0.56 rpy=0 -0.523598775598 0.17 -> xyz=-0.1 -0.03 0.56 rpy=0 -1.57079632679 0.17
- joint middle_kinect_base_to_kinect2: origin xyz=0.25 0 0 rpy=-0.785398163397 0 -1.57079632679 -> xyz=0.25 0 0 rpy=-1.57079632679 0 -1.57079632679
- joint yumi_to_middle_kinect_base: origin xyz=0.05 0 0.56 rpy=0 -0.523598775598 0 -> xyz=-0.1 0 0.56 rpy=0 -1.57079632679 0

File: ridgeback_yumi_description/urdf/ridgeback_yumi.urdf.xacro (robot description, xacro)
@@ -37,4 +37,5 @@
   <xacro:property name="yumi_height" value="0.25" />
   <xacro:property name="kinect_zrotation_fix" value="${- PI / 2.0}" />
+  <xacro:property name="kinect_base_pitch" value="${ -PI/2.0 }" />
   <joint name="ridgeback_base_to_pedestal" type="fixed">
     <origin rpy="0 0 ${PI}" xyz="${pedestal_offset_x} 0 ${pedestal_height}" />
@@ -102,20 +103,20 @@
     <parent link="yumi_base_link" />
     <child link="right_kinect_base" />
-    <origin rpy="0 ${-PI/6} 0.17" xyz="0.1 -0.03 0.56" />
+    <origin rpy="0 ${-PI/2} 0.17" xyz="-0.1 -0.03 0.56" />
   </joint>
   <joint name="kinect2_to_left_kinect_base" type="fixed">
     <parent link="yumi_base_link" />
     <child link="left_kinect_base" />
-    <origin rpy="0 ${-PI/6} -0.17" xyz="0.1 0.03 0.56" />
+    <origin rpy="0 ${-PI/2} -0.17" xyz="-0.1 0.03 0.56" />
   </joint>
   <joint name="yumi_to_middle_kinect_base" type="fixed">
     <parent link="yumi_base_link" />
     <child link="middle_kinect_base" />
-    <origin rpy="0 ${-PI/6} 0" xyz="0.05 0 0.56" />
+    <origin rpy="0 ${kinect_base_pitch} 0" xyz="-0.1 0 0.56" />
   </joint>
   <joint name="middle_kinect_base_to_kinect2" type="fixed">
     <parent link="middle_kinect_base" />
     <child link="kinect2" />
-    <origin rpy="${-PI/4} 0 ${kinect_zrotation_fix}" xyz="0.25 0 0" />
+    <origin rpy="${-PI/2} 0 ${kinect_zrotation_fix}" xyz="0.25 0 0" />
   </joint>
 </robot>

Commit message: Calibration of Optoforce 6axis FT sensors

File: ridgeback_yumi_description/urdf/ridgeback_yumi.urdf (robot description, URDF)
Before this commit: robot ridgeback_yumi, 48 links, 47 joints
Joints:
- joint optodaq_l_sensor_link_joint: origin xyz=0 0 0.033 rpy=0 0 3.14159265359 -> xyz=0 0 -0.033 rpy=3.14159265359 0.0 0.785398163397
- joint optodaq_r_sensor_link_joint: origin xyz=0 0 0.033 rpy=0 0 3.14159265359 -> xyz=0 0 -0.033 rpy=3.14159265359 0.0 0.785398163397
- joint yumi_link_7_l_joint: origin xyz=0 0 0.033 rpy=0 0 3.14159265359 -> xyz=0 0 0.033 rpy=0 3.14159265359 -0.785398163397
- joint yumi_link_7_r_joint: origin xyz=0 0 0.033 rpy=0 0 3.14159265359 -> xyz=0 0 0.033 rpy=0 3.14159265359 -0.785398163397

File: ridgeback_yumi_description/urdf/ridgeback_yumi.urdf.xacro (robot description, xacro)
@@ -19,16 +19,16 @@
   </xacro:yumi>
   <xacro:yumi_optodaq_sensor name="optodaq_r" parent="yumi_link_7_r">
-      <origin xyz="0 0 0.033" rpy="0 ${PI} ${PI}" />
+      <origin xyz="0 0 0.033" rpy="0 ${PI} ${-PI/4}" />
   </xacro:yumi_optodaq_sensor>
   <xacro:yumi_optodaq_sensor name="optodaq_l" parent="yumi_link_7_l">
-    <origin xyz="0 0 0.033" rpy="0 ${PI} -0.7" />
+	  <origin xyz="0 0 0.033" rpy="0 ${PI} ${-PI/4}" />
   </xacro:yumi_optodaq_sensor>
   <!--right gripper-->
   <xacro:yumi_servo_gripper name="gripper_r" hardware_interface="hardware_interface/EffortJointInterface" parent="optodaq_r_sensor_link">
-    <origin xyz="0 0 -0.033" rpy="0 ${-PI} ${PI}" />
+    <origin xyz="0 0 -0.033" rpy="${PI} 0.0 ${PI/4}" />
   </xacro:yumi_servo_gripper>
   <!--left gripper-->
   <xacro:yumi_servo_gripper name="gripper_l" hardware_interface="hardware_interface/EffortJointInterface" parent="optodaq_l_sensor_link">
-    <origin xyz="0 0 -0.033" rpy="0 ${-PI} ${PI}" />
+    <origin xyz="0 0 -0.033" rpy="${PI} 0.0 ${PI/4}" />
   </xacro:yumi_servo_gripper>
   <xacro:property name="pedestal_height" value="0.28" />
