Commit message: Fixing some things after trying out the package on the real robots

File: ridgeback_yumi_description/urdf/ridgeback_yumi.urdf.xacro (robot description, xacro)
@@ -12,8 +12,8 @@
   <!-- Import Gazebo plugins -->
   <xacro:include filename="$(find yumi_description)/urdf/Gazebo/gazebo.urdf.xacro"/>
-  <!-- Fix to world just for testing -->
-  <link name="world"/>
+  <!-- Fix to world just for testing
+  <link name="world"/> -->
   <!--yumi-->
-  <xacro:yumi name="yumi" hardware_interface="hardware_interface/$(arg arms_interface)" parent="world">
+  <xacro:yumi name="yumi" hardware_interface="hardware_interface/$(arg arms_interface)" parent="base_link">
     <origin xyz="0 0 0.1" rpy="0 0 0" />
   </xacro:yumi>
@@ -26,11 +26,10 @@
     <origin xyz="0 0 0.007" rpy="0 0 ${PI}" />
   </xacro:yumi_servo_gripper>
-  <xacro:property name="pedestal_height" value="-0.54" />
-  <xacro:property name="pedestal_diameter" value="0.203" />
-  <xacro:property name="pedestal_offset_x" value="-0.30" />
+  <xacro:property name="pedestal_height" value="0.54" />
+  <xacro:property name="pedestal_offset_x" value="0.30" />
   <joint name="ridgeback_base_to_yumi" type="fixed">
     <origin rpy="0 0 0" xyz="${pedestal_offset_x} 0 ${pedestal_height}" />
-    <parent link="yumi_body" />
-    <child link="base_link" />
+    <parent link="base_link" />
+    <child link="yumi_body" />
   </joint>
 </robot>

Commit message: Added the pedestal mesh and corresponding joint, links and transform in the URDF file

File: ridgeback_yumi_description/urdf/ridgeback_yumi.urdf.xacro (robot description, xacro)
@@ -26,9 +26,25 @@
     <origin xyz="0 0 0.007" rpy="0 0 ${PI}" />
   </xacro:yumi_servo_gripper>
-  <xacro:property name="pedestal_height" value="0.54" />
-  <xacro:property name="pedestal_offset_x" value="0.30" />
-  <joint name="ridgeback_base_to_yumi" type="fixed">
-    <origin rpy="0 0 0" xyz="${pedestal_offset_x} 0 ${pedestal_height}" />
+  <xacro:property name="pedestal_height" value="0.28" />
+  <xacro:property name="pedestal_offset_x" value="0.32" />
+  <xacro:property name="yumi_offset_x" value="0.06" />
+  <xacro:property name="yumi_height" value="0.25" />
+  <joint name="ridgeback_base_to_pedestal" type="fixed">
+    <origin rpy="0 0 ${PI}" xyz="${pedestal_offset_x} 0 ${pedestal_height}" />
     <parent link="base_link" />
+    <child link="yumi_pedestal" />
+  </joint>
+  <link name="yumi_pedestal">
+    <visual>
+      <origin xyz="0 0 0" rpy="0 0 ${PI}" />
+      <geometry>
+        <mesh filename="package://ridgeback_yumi_description/meshes/IRB14000_mount.stl"/>
+      </geometry>
+      <material name="black" />
+    </visual>
+  </link>
+  <joint name="pedestal_to_yumi" type="fixed">
+    <origin rpy="0 0 ${PI}" xyz="${yumi_offset_x} 0 ${yumi_height}" />
+    <parent link="yumi_pedestal" />
     <child link="yumi_body" />
   </joint>

Commit message: Updated the URDF to satisfy our new YuMi URDF structure

File: ridgeback_yumi_description/urdf/ridgeback_yumi.urdf.xacro (robot description, xacro)
@@ -12,8 +12,6 @@
   <!-- Import Gazebo plugins -->
   <xacro:include filename="$(find yumi_description)/urdf/Gazebo/gazebo.urdf.xacro"/>
-  <!-- Fix to world just for testing
-  <link name="world"/> -->
   <!--yumi-->
-  <xacro:yumi name="yumi" hardware_interface="hardware_interface/VelocityJointInterface" parent="base_link">
+  <xacro:yumi name="yumi" hardware_interface="hardware_interface/VelocityJointInterface" parent="yumi_pedestal">
     <origin xyz="0 0 0.1" rpy="0 0 0" />
   </xacro:yumi>
@@ -36,4 +34,11 @@
   </joint>
   <link name="yumi_pedestal">
+    <collision>
+      <origin xyz="0 0 0" rpy="0 0 ${PI}" />
+      <geometry>
+        <mesh filename="package://ridgeback_yumi_description/meshes/IRB14000_mount.stl"/>
+      </geometry>
+      <material name="black" />
+    </collision>
     <visual>
       <origin xyz="0 0 0" rpy="0 0 ${PI}" />
@@ -47,5 +52,5 @@
     <origin rpy="0 0 ${PI}" xyz="${yumi_offset_x} 0 ${yumi_height}" />
     <parent link="yumi_pedestal" />
-    <child link="yumi_body" />
+    <child link="yumi_base_link" />
   </joint>
 </robot>

Commit message: Fixing some bugs related to the optodaq sub-package

File: ridgeback_yumi_description/urdf/ridgeback_yumi.urdf.xacro (robot description, xacro)
@@ -10,4 +10,6 @@
   <!--Import the yumi servo gripper macro -->
   <xacro:include filename="$(find yumi_description)/urdf/Grippers/yumi_servo_gripper.xacro"/>
+  <!--Import the yumi optodaq sensors macro -->
+  <xacro:include filename="$(find yumi_description)/urdf/Extras/yumi_optodaq_sensors.xacro"/>
   <!-- Import Gazebo plugins -->
   <xacro:include filename="$(find yumi_description)/urdf/Gazebo/gazebo.urdf.xacro"/>
@@ -16,11 +18,17 @@
     <origin xyz="0 0 0.1" rpy="0 0 0" />
   </xacro:yumi>
+  <xacro:yumi_optodaq_sensor name="optodaq_r" parent="yumi_link_7_r">
+      <origin xyz="0 0 0.033" rpy="0 0 ${PI}" />
+  </xacro:yumi_optodaq_sensor>
+  <xacro:yumi_optodaq_sensor name="optodaq_l" parent="yumi_link_7_l">
+    <origin xyz="0 0 0.033" rpy="0 0 ${PI}" />
+  </xacro:yumi_optodaq_sensor>
   <!--right gripper-->
-  <xacro:yumi_servo_gripper name="gripper_r" hardware_interface="hardware_interface/EffortJointInterface" parent="yumi_link_7_r">
-    <origin xyz="0 0 0.007" rpy="0 0 ${PI}" />
+  <xacro:yumi_servo_gripper name="gripper_r" hardware_interface="hardware_interface/EffortJointInterface" parent="optodaq_r_sensor_link">
+    <origin xyz="0 0 0.033" rpy="0 0 ${PI}" />
   </xacro:yumi_servo_gripper>
   <!--left gripper-->
-  <xacro:yumi_servo_gripper name="gripper_l" hardware_interface="hardware_interface/EffortJointInterface" parent="yumi_link_7_l">
-    <origin xyz="0 0 0.007" rpy="0 0 ${PI}" />
+  <xacro:yumi_servo_gripper name="gripper_l" hardware_interface="hardware_interface/EffortJointInterface" parent="optodaq_l_sensor_link">
+    <origin xyz="0 0 0.033" rpy="0 0 ${PI}" />
   </xacro:yumi_servo_gripper>
   <xacro:property name="pedestal_height" value="0.28" />

Commit message: Full MoveIt! config for ridgeback_yumi. Also added a simple launch file for exporting the URDF, and cleaned the sub-package ridgeback_yumi_description a bit

File: ridgeback_yumi_description/urdf/ridgeback_yumi.urdf.xacro (robot description, xacro)
@@ -36,4 +36,5 @@
   <xacro:property name="yumi_offset_x" value="0.06" />
   <xacro:property name="yumi_height" value="0.25" />
+  <xacro:property name="kinect_zrotation_fix" value="${- PI / 2.0}" />
   <joint name="ridgeback_base_to_pedestal" type="fixed">
     <origin rpy="0 0 ${PI}" xyz="${pedestal_offset_x} 0 ${pedestal_height}" />
@@ -62,3 +63,59 @@
     <child link="yumi_base_link" />
   </joint>
+  <link name="kinect2">
+    <visual>
+      <origin xyz="0 0 0" rpy="0 0 0" />
+      <geometry>
+        <mesh scale="0.001 0.001 0.001" filename="package://yumi_description/meshes/accesories/KinectXboxOne.stl"/>
+      </geometry>
+      <material name="Black" />
+    </visual>
+  </link>
+  <link name="left_kinect_base">
+      <visual>
+        <origin xyz="0 0 0" rpy="0 0 0" />
+        <geometry>
+          <box size="0.4 0.02 0.02" />
+        </geometry>
+        <material name="Grey" />
+      </visual>
+  </link>
+  <link name="right_kinect_base">
+      <visual>
+        <origin xyz="0 0 0" rpy="0 0 0" />
+        <geometry>
+          <box size="0.4 0.02 0.02" />
+        </geometry>
+        <material name="Grey" />
+      </visual>
+  </link>
+  <link name="middle_kinect_base">
+      <visual>
+        <origin xyz="0 0 0" rpy="0 0 0" />
+        <geometry>
+          <box size="0.4 0.02 0.02" />
+        </geometry>
+        <material name="Grey" />
+      </visual>
+  </link>
+   <joint name="kinect2_to_right_kinect_base" type="fixed">
+    <parent link="yumi_base_link" />
+    <child link="right_kinect_base" />
+    <origin rpy="0 ${-PI/6} 0.17" xyz="0.1 -0.03 0.56" />
+  </joint>
+  <joint name="kinect2_to_left_kinect_base" type="fixed">
+    <parent link="yumi_base_link" />
+    <child link="left_kinect_base" />
+    <origin rpy="0 ${-PI/6} -0.17" xyz="0.1 0.03 0.56" />
+  </joint>
+  <joint name="yumi_to_middle_kinect_base" type="fixed">
+    <parent link="yumi_base_link" />
+    <child link="middle_kinect_base" />
+    <origin rpy="0 ${-PI/6} 0" xyz="0.05 0 0.56" />
+  </joint>
+  <joint name="middle_kinect_base_to_kinect2" type="fixed">
+    <parent link="middle_kinect_base" />
+    <child link="kinect2" />
+    <origin rpy="${-PI/4} 0 ${kinect_zrotation_fix}" xyz="0.25 0 0" />
+  </joint>
 </robot>

Commit message: Small fix in the URDF towards the force-torque sensor calibration

File: ridgeback_yumi_description/urdf/ridgeback_yumi.urdf.xacro (robot description, xacro)
@@ -19,16 +19,16 @@
   </xacro:yumi>
   <xacro:yumi_optodaq_sensor name="optodaq_r" parent="yumi_link_7_r">
-      <origin xyz="0 0 0.033" rpy="0 0 ${PI}" />
+      <origin xyz="0 0 0.033" rpy="0 ${PI} ${PI}" />
   </xacro:yumi_optodaq_sensor>
   <xacro:yumi_optodaq_sensor name="optodaq_l" parent="yumi_link_7_l">
-    <origin xyz="0 0 0.033" rpy="0 0 ${PI}" />
+    <origin xyz="0 0 0.033" rpy="0 ${PI} -0.7" />
   </xacro:yumi_optodaq_sensor>
   <!--right gripper-->
   <xacro:yumi_servo_gripper name="gripper_r" hardware_interface="hardware_interface/EffortJointInterface" parent="optodaq_r_sensor_link">
-    <origin xyz="0 0 0.033" rpy="0 0 ${PI}" />
+    <origin xyz="0 0 -0.033" rpy="0 ${-PI} ${PI}" />
   </xacro:yumi_servo_gripper>
   <!--left gripper-->
   <xacro:yumi_servo_gripper name="gripper_l" hardware_interface="hardware_interface/EffortJointInterface" parent="optodaq_l_sensor_link">
-    <origin xyz="0 0 0.033" rpy="0 0 ${PI}" />
+    <origin xyz="0 0 -0.033" rpy="0 ${-PI} ${PI}" />
   </xacro:yumi_servo_gripper>
   <xacro:property name="pedestal_height" value="0.28" />

Commit message: Changed the orientation and parents of Optoforce sensors link to the correct one, specified by vendor

File: ridgeback_yumi_description/urdf/ridgeback_yumi.urdf.xacro (robot description, xacro)
@@ -14,21 +14,22 @@
   <!-- Import Gazebo plugins -->
   <xacro:include filename="$(find yumi_description)/urdf/Gazebo/gazebo.urdf.xacro"/>
-  <!--yumi-->
+  <!-- yumi -->
   <xacro:yumi name="yumi" hardware_interface="hardware_interface/VelocityJointInterface" parent="yumi_pedestal">
     <origin xyz="0 0 0.1" rpy="0 0 0" />
   </xacro:yumi>
+  <!-- Optoforce F/T sensors -->
   <xacro:yumi_optodaq_sensor name="optodaq_r" parent="yumi_link_7_r">
-      <origin xyz="0 0 0.033" rpy="0 ${PI} ${-PI/4}" />
+      <origin xyz="0 0 0.033" rpy="0 0 ${-PI/2}" />
   </xacro:yumi_optodaq_sensor>
   <xacro:yumi_optodaq_sensor name="optodaq_l" parent="yumi_link_7_l">
-	  <origin xyz="0 0 0.033" rpy="0 ${PI} ${-PI/4}" />
+    <origin xyz="0 0 0.033" rpy="0 0 ${-PI/2}" />
   </xacro:yumi_optodaq_sensor>
-  <!--right gripper-->
+  <!-- Right gripper -->
   <xacro:yumi_servo_gripper name="gripper_r" hardware_interface="hardware_interface/EffortJointInterface" parent="optodaq_r_sensor_link">
-    <origin xyz="0 0 -0.033" rpy="${PI} 0.0 ${PI/4}" />
+    <origin xyz="0 0 0.033" rpy="0 0.0 ${PI/4}" />
   </xacro:yumi_servo_gripper>
-  <!--left gripper-->
+  <!-- Left gripper -->
   <xacro:yumi_servo_gripper name="gripper_l" hardware_interface="hardware_interface/EffortJointInterface" parent="optodaq_l_sensor_link">
-    <origin xyz="0 0 -0.033" rpy="${PI} 0.0 ${PI/4}" />
+    <origin xyz="0 0 0.033" rpy="0 0.0 ${PI/4}" />
   </xacro:yumi_servo_gripper>
   <xacro:property name="pedestal_height" value="0.28" />

Commit message: Fixed cylinder (sensor) length to match the new mounts

File: ridgeback_yumi_description/urdf/ridgeback_yumi.urdf.xacro (robot description, xacro)
@@ -20,16 +20,16 @@
   <!-- Optoforce F/T sensors -->
   <xacro:yumi_optodaq_sensor name="optodaq_r" parent="yumi_link_7_r">
-      <origin xyz="0 0 0.033" rpy="0 0 ${-PI/2}" />
+      <origin xyz="0 0 0.0445" rpy="0 0 ${-PI/2}" />
   </xacro:yumi_optodaq_sensor>
   <xacro:yumi_optodaq_sensor name="optodaq_l" parent="yumi_link_7_l">
-    <origin xyz="0 0 0.033" rpy="0 0 ${-PI/2}" />
+    <origin xyz="0 0 0.0445" rpy="0 0 ${-PI/2}" />
   </xacro:yumi_optodaq_sensor>
   <!-- Right gripper -->
   <xacro:yumi_servo_gripper name="gripper_r" hardware_interface="hardware_interface/EffortJointInterface" parent="optodaq_r_sensor_link">
-    <origin xyz="0 0 0.033" rpy="0 0.0 ${PI/4}" />
+    <origin xyz="0 0 0.0445" rpy="0 0.0 ${PI/4}" />
   </xacro:yumi_servo_gripper>
   <!-- Left gripper -->
   <xacro:yumi_servo_gripper name="gripper_l" hardware_interface="hardware_interface/EffortJointInterface" parent="optodaq_l_sensor_link">
-    <origin xyz="0 0 0.033" rpy="0 0.0 ${PI/4}" />
+    <origin xyz="0 0 0.0445" rpy="0 0.0 ${PI/4}" />
   </xacro:yumi_servo_gripper>
   <xacro:property name="pedestal_height" value="0.28" />

Commit message: Updated sensor tf values

File: ridgeback_yumi_description/urdf/ridgeback_yumi.urdf.xacro (robot description, xacro)
@@ -20,8 +20,8 @@
   <!-- Optoforce F/T sensors -->
   <xacro:yumi_optodaq_sensor name="optodaq_r" parent="yumi_link_7_r">
-      <origin xyz="0 0 0.0445" rpy="0 0 ${-PI/2}" />
+      <origin xyz="0 0 0.0445" rpy="0 0 0" />
   </xacro:yumi_optodaq_sensor>
   <xacro:yumi_optodaq_sensor name="optodaq_l" parent="yumi_link_7_l">
-    <origin xyz="0 0 0.0445" rpy="0 0 ${-PI/2}" />
+    <origin xyz="0 0 0.0445" rpy="0 0 0" />
   </xacro:yumi_optodaq_sensor>
   <!-- Right gripper -->
